File: Clock/Clock.kicad_pcb (KiCad board)
At the start: 2 copper layers, 200 x 100 mm, 64 parts, among them J1 Conn buss, J10 Conn_buss, J11 Conn_buss, J12 Conn_buss, J13 Register_A-1,2 LED Conn, J14 Register_B-1,2 LED Conn, J15 Program Counter LED Conn, J16 Memory Address Reg LED Conn, J17 Instruction Reg LED Conn, J18 Conn_01x02_Pin, J19 Conn_02x04_Top_Bottom, J2 USB4125-GF-A, J3 Fuse-Block, J4 Conn buss, J5 Conn_buss, J6 Conn_buss, J7 Conn_buss, J8 Conn_buss, J9 Conn_buss, SW1 SW_CLK_mono, SW2 SW_Select_Mon/Ast, SW3 SW_SPST, SW4 SW_Select_Oscilator, U1 NE555P, U10 CD74HCT153E, U2 NE555P, U3 NE555P, U4 74LS04, U5 74LS08, U6 CD74HCT14E, U7 NE555P, Y1 ECS-100AX-010

Commit message: Routed bus connector
Parts:
- removed J13: Register_A-1,2 LED Conn, Connector_PinHeader_2.54mm:PinHeader_2x08_P2.54mm_Vertical
- removed J14: Register_B-1,2 LED Conn, Connector_PinHeader_2.54mm:PinHeader_2x08_P2.54mm_Vertical
- removed J15: Program Counter LED Conn, Connector_PinHeader_2.54mm:PinHeader_2x08_P2.54mm_Vertical
- removed J16: Memory Address Reg LED Conn, Connector_PinHeader_2.54mm:PinHeader_2x08_P2.54mm_Vertical
- removed J17: Instruction Reg LED Conn, Connector_PinHeader_2.54mm:PinHeader_2x08_P2.54mm_Vertical
- C10: footprint Capacitor_THT:C_Radial_D5.0mm_H7.0mm_P2.00mm -> Capacitor_THT:CP_Radial_D5.0mm_P2.00mm
- moved U6 363.5 mm to (-61.0, 44.3)
- moved C14 352.0 mm to (-75.6, 72.7)
- moved C15 351.2 mm to (-74.7, 66.1)
- moved C17 338.0 mm to (-60.9, 59.7)
- moved C5 331.4 mm to (-62.2, 31.6)
- moved C13 317.9 mm to (-46.3, 60.7)
- moved C4 309.6 mm to (-40.1, 28.6)
- moved C12 304.6 mm to (-32.9, 56.6)
- moved C3 295.7 mm to (-26.6, 28.6)
- moved C11 286.1 mm to (-14.7, 57.2)
- moved C2 278.0 mm to (-9.51, 30.2), turned to 180 degrees
- moved C16 256.9 mm to (19.6, 80.3)
- moved Y1 246.5 mm to (27.9, 91.4)
- moved U7 129.8 mm to (-62.9, 64.8)
- moved J12 118.4 mm to (75.6, 113.4)
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Connections:
- net AS renamed /MEM_RD_N
- net B0I renamed /MEM_WR_N
- net B0O renamed /BUS_SRC0
- net B1I renamed /BUS_SRC2
- net B1O renamed /BUS_SRC1
- net CYI renamed /A3
- net CYO renamed /A4
- net ECOMP renamed /ALU_S0
- net EM renamed /BUS_DST1
- net EO renamed /BUS_DST0
- net ES0 renamed /BUS_DST2
- net ES2 renamed /A_SEL
- net ES3 renamed /B_SEL
- net Ex0I renamed /ALU_S2
- net Ex0O renamed /ALU_S3
- net Ex10 renamed /ALU_CIN_N
- net Ex1I renamed /ALU_M
- net OI renamed /ALU_S1
- net SPI renamed /ALU_COUT
- J1 pad 1: MI -> /D0
- J1 pad 10: A1I -> GND
- J1 pad 16: BS -> GND
- J1 pad 2: RI -> /D1
- J1 pad 20: ES1 -> GND
- J1 pad 3: RO -> /D2
- J1 pad 30: SPO -> +5V
- J1 pad 31: HLT -> GND
- J1 pad 32: GND -> /A0
- J1 pad 33: CLK -> /A1
- J1 pad 34: GND -> /A2
- J1 pad 37: Bus C0 -> /A5
- J1 pad 38: Bus C1 -> /A6
- J1 pad 39: Bus C2 -> /A7
- J1 pad 4: CO -> /D3
- J1 pad 40: Bus C3 -> +5V
- J1 pad 41: Bus C4 -> /A8
- J1 pad 42: Bus C5 -> /A9
- J1 pad 43: Bus C6 -> /A10
- J1 pad 44: Bus C7 -> /A11
- J1 pad 45: /Inst_Reg_LED1 -> /A12
- J1 pad 46: /Inst_Reg_LED2 -> /A13
- J1 pad 47: /Inst_Reg_LED3 -> /A14
- J1 pad 48: /Inst_Reg_LED4 -> /A15
- J1 pad 49: /Inst_Reg_LED5 -> GND
- J1 pad 5: CE -> /D4
- J1 pad 50: /Inst_Reg_LED6 -> GND
- J1 pad 51: /Inst_Reg_LED7 -> /FLAGS_WE
- J1 pad 52: /Inst_Reg_LED8 -> /PC_INC
- J1 pad 53: /Inst_Reg_LED9 -> /PC_TO_MAR
- J1 pad 54: /Inst_Reg_LED10 -> /SP_INC
- J1 pad 55: /Inst_Reg_LED11 -> /SP_DEC
- J1 pad 56: /Inst_Reg_LED12 -> /RESET_N
- J1 pad 57: /Inst_Reg_LED13 -> /WAIT_N
- J1 pad 58: /Inst_Reg_LED14 -> /IRQ_N
- J1 pad 59: /Inst_Reg_LED15 -> /Unused
- J1 pad 6: J -> /D5
- J1 pad 60: /Inst_Reg_LED16 -> +5V
- J1 pad 61: +5V -> GND
- J1 pad 62: GND -> CLK
- J1 pad 7: A0I -> /D6
- J1 pad 8: A0O -> /D7
- J1 pad 9: A1O -> +5V
- J10 pad 1: MI -> /D0
- J10 pad 10: A1I -> GND
- J10 pad 16: BS -> GND
- J10 pad 2: RI -> /D1
- J10 pad 20: ES1 -> GND
- J10 pad 3: RO -> /D2
- J10 pad 30: SPO -> +5V
- J10 pad 31: HLT -> GND
- J10 pad 32: GND -> /A0
- J10 pad 33: CLK -> /A1
- J10 pad 34: GND -> /A2
- J10 pad 37: Bus C0 -> /A5
- J10 pad 38: Bus C1 -> /A6
- J10 pad 39: Bus C2 -> /A7
- J10 pad 4: CO -> /D3
- J10 pad 40: Bus C3 -> +5V
- J10 pad 41: Bus C4 -> /A8
- J10 pad 42: Bus C5 -> /A9
- J10 pad 43: Bus C6 -> /A10
- J10 pad 44: Bus C7 -> /A11
- J10 pad 45: unconnected-(J10-Pad45) -> /A12
- J10 pad 46: unconnected-(J10-Pad46) -> /A13
- J10 pad 47: unconnected-(J10-Pad47) -> /A14
- J10 pad 48: unconnected-(J10-Pad48) -> /A15
- J10 pad 49: unconnected-(J10-Pad49) -> GND
- J10 pad 5: CE -> /D4
- J10 pad 50: unconnected-(J10-Pad50) -> GND
- J10 pad 51: unconnected-(J10-Pad51) -> /FLAGS_WE
- J10 pad 52: unconnected-(J10-Pad52) -> /PC_INC
- J10 pad 53: unconnected-(J10-Pad53) -> /PC_TO_MAR
- J10 pad 54: unconnected-(J10-Pad54) -> /SP_INC
- J10 pad 55: unconnected-(J10-Pad55) -> /SP_DEC
- J10 pad 56: unconnected-(J10-Pad56) -> /RESET_N
- J10 pad 57: unconnected-(J10-Pad57) -> /WAIT_N
- J10 pad 58: unconnected-(J10-Pad58) -> /IRQ_N
- J10 pad 59: unconnected-(J10-Pad59) -> /Unused
- J10 pad 6: J -> /D5
- J10 pad 60: unconnected-(J10-Pad60) -> +5V
- J10 pad 61: +5V -> GND
- J10 pad 62: GND -> CLK
- J10 pad 7: A0I -> /D6
- J10 pad 8: A0O -> /D7
- J10 pad 9: A1O -> +5V
- J11 pad 1: MI -> /D0
- J11 pad 10: A1I -> GND
- J11 pad 16: BS -> GND
- J11 pad 2: RI -> /D1
- J11 pad 20: ES1 -> GND
- J11 pad 3: RO -> /D2
- J11 pad 30: SPO -> +5V
- J11 pad 31: HLT -> GND
- J11 pad 32: GND -> /A0
- J11 pad 33: CLK -> /A1
- J11 pad 34: GND -> /A2
- J11 pad 37: Bus C0 -> /A5
- J11 pad 38: Bus C1 -> /A6
- J11 pad 39: Bus C2 -> /A7
- J11 pad 4: CO -> /D3
- J11 pad 40: Bus C3 -> +5V
- J11 pad 41: Bus C4 -> /A8
- J11 pad 42: Bus C5 -> /A9
- J11 pad 43: Bus C6 -> /A10
- J11 pad 44: Bus C7 -> /A11
- J11 pad 45: /RegA_LED1 -> /A12
- J11 pad 46: /RegA_LED2 -> /A13
- J11 pad 47: /RegA_LED3 -> /A14
- J11 pad 48: /RegA_LED4 -> /A15
- J11 pad 49: /RegA_LED5 -> GND
- J11 pad 5: CE -> /D4
- J11 pad 50: /RegA_LED6 -> GND
- J11 pad 51: /RegA_LED7 -> /FLAGS_WE
- J11 pad 52: /RegA_LED8 -> /PC_INC
- J11 pad 53: /RegA_LED9 -> /PC_TO_MAR
- J11 pad 54: /RegA_LED10 -> /SP_INC
- J11 pad 55: /RegA_LED11 -> /SP_DEC
- J11 pad 56: /RegA_LED12 -> /RESET_N
- J11 pad 57: /RegA_LED13 -> /WAIT_N
- J11 pad 58: /RegA_LED14 -> /IRQ_N
- J11 pad 59: /RegA_LED15 -> /Unused
- J11 pad 6: J -> /D5
- J11 pad 60: /RegA_LED16 -> +5V
- J11 pad 61: +5V -> GND
- J11 pad 62: GND -> CLK
- J11 pad 7: A0I -> /D6
- J11 pad 8: A0O -> /D7
- J11 pad 9: A1O -> +5V
- J12 pad 1: MI -> /D0
- J12 pad 10: A1I -> GND
- J12 pad 16: BS -> GND
- J12 pad 2: RI -> /D1
- J12 pad 20: ES1 -> GND
- J12 pad 3: RO -> /D2
- J12 pad 30: SPO -> +5V
- J12 pad 31: HLT -> GND
- J12 pad 32: GND -> /A0
- J12 pad 33: CLK -> /A1
- J12 pad 34: GND -> /A2
- J12 pad 37: Bus C0 -> /A5
- J12 pad 38: Bus C1 -> /A6
- J12 pad 39: Bus C2 -> /A7
- J12 pad 4: CO -> /D3
- J12 pad 40: Bus C3 -> +5V
- J12 pad 41: Bus C4 -> /A8
- J12 pad 42: Bus C5 -> /A9
- J12 pad 43: Bus C6 -> /A10
- J12 pad 44: Bus C7 -> /A11
- J12 pad 45: unconnected-(J12-Pad45) -> /A12
- J12 pad 46: unconnected-(J12-Pad46) -> /A13
- J12 pad 47: unconnected-(J12-Pad47) -> /A14
- J12 pad 48: unconnected-(J12-Pad48) -> /A15
- J12 pad 49: unconnected-(J12-Pad49) -> GND
- J12 pad 5: CE -> /D4
- J12 pad 50: unconnected-(J12-Pad50) -> GND
- J12 pad 51: unconnected-(J12-Pad51) -> /FLAGS_WE
- J12 pad 52: unconnected-(J12-Pad52) -> /PC_INC
- J12 pad 53: unconnected-(J12-Pad53) -> /PC_TO_MAR
- J12 pad 54: unconnected-(J12-Pad54) -> /SP_INC
- J12 pad 55: unconnected-(J12-Pad55) -> /SP_DEC
- J12 pad 56: unconnected-(J12-Pad56) -> /RESET_N
- J12 pad 57: unconnected-(J12-Pad57) -> /WAIT_N
- J12 pad 58: unconnected-(J12-Pad58) -> /IRQ_N
- J12 pad 59: unconnected-(J12-Pad59) -> /Unused
- J12 pad 6: J -> /D5
- J12 pad 60: unconnected-(J12-Pad60) -> +5V
- J12 pad 61: +5V -> GND
- J12 pad 62: GND -> CLK
- J12 pad 7: A0I -> /D6
- J12 pad 8: A0O -> /D7
- J12 pad 9: A1O -> +5V
- J19 pad 1: Bus C0 -> /D0
- J19 pad 2: Bus C1 -> /D1
- J19 pad 3: Bus C2 -> /D2
- J19 pad 4: Bus C3 -> /D3
- J19 pad 5: Bus C4 -> /D4
- J19 pad 6: Bus C5 -> /D5
- J19 pad 7: Bus C6 -> /D6
- J19 pad 8: Bus C7 -> /D7
- J4 pad 1: MI -> /D0
- J4 pad 10: A1I -> GND
- J4 pad 16: BS -> GND
- J4 pad 2: RI -> /D1
- J4 pad 20: ES1 -> GND
- J4 pad 3: RO -> /D2
- J4 pad 30: SPO -> +5V
- J4 pad 31: HLT -> GND
- J4 pad 32: GND -> /A0
- J4 pad 33: CLK -> /A1
- J4 pad 34: GND -> /A2
- J4 pad 37: Bus C0 -> /A5
- J4 pad 38: Bus C1 -> /A6
- J4 pad 39: Bus C2 -> /A7
- J4 pad 4: CO -> /D3
- J4 pad 40: Bus C3 -> +5V
- J4 pad 41: Bus C4 -> /A8
- J4 pad 42: Bus C5 -> /A9
- J4 pad 43: Bus C6 -> /A10
- J4 pad 44: Bus C7 -> /A11
- J4 pad 45: unconnected-(J4-Pad45) -> /A12
- J4 pad 46: unconnected-(J4-Pad46) -> /A13
- J4 pad 47: unconnected-(J4-Pad47) -> /A14
- J4 pad 48: unconnected-(J4-Pad48) -> /A15
- J4 pad 49: unconnected-(J4-Pad49) -> GND
- J4 pad 5: CE -> /D4
- J4 pad 50: unconnected-(J4-Pad50) -> GND
- J4 pad 51: unconnected-(J4-Pad51) -> /FLAGS_WE
- J4 pad 52: unconnected-(J4-Pad52) -> /PC_INC
- J4 pad 53: unconnected-(J4-Pad53) -> /PC_TO_MAR
- J4 pad 54: unconnected-(J4-Pad54) -> /SP_INC
- J4 pad 55: unconnected-(J4-Pad55) -> /SP_DEC
- J4 pad 56: unconnected-(J4-Pad56) -> /RESET_N
- J4 pad 57: unconnected-(J4-Pad57) -> /WAIT_N
- J4 pad 58: unconnected-(J4-Pad58) -> /IRQ_N
- J4 pad 59: unconnected-(J4-Pad59) -> /Unused
- J4 pad 6: J -> /D5
- J4 pad 60: unconnected-(J4-Pad60) -> +5V
- J4 pad 61: +5V -> GND
- J4 pad 62: GND -> CLK
- J4 pad 7: A0I -> /D6
- J4 pad 8: A0O -> /D7
- J4 pad 9: A1O -> +5V
- J5 pad 1: MI -> /D0
- J5 pad 10: A1I -> GND
- J5 pad 16: BS -> GND
- J5 pad 2: RI -> /D1
- J5 pad 20: ES1 -> GND
- J5 pad 3: RO -> /D2
- J5 pad 30: SPO -> +5V
- J5 pad 31: HLT -> GND
- J5 pad 32: GND -> /A0
- J5 pad 33: CLK -> /A1
- J5 pad 34: GND -> /A2
- J5 pad 37: Bus C0 -> /A5
- J5 pad 38: Bus C1 -> /A6
- J5 pad 39: Bus C2 -> /A7
- J5 pad 4: CO -> /D3
- J5 pad 40: Bus C3 -> +5V
- J5 pad 41: Bus C4 -> /A8
- J5 pad 42: Bus C5 -> /A9
- J5 pad 43: Bus C6 -> /A10
- J5 pad 44: Bus C7 -> /A11
- J5 pad 45: /Mem_addreg1 -> /A12
- J5 pad 46: /Mem_addreg2 -> /A13
- J5 pad 47: /Mem_addreg3 -> /A14
- J5 pad 48: /Mem_addreg4 -> /A15
- J5 pad 49: /Mem_addreg5 -> GND
- J5 pad 5: CE -> /D4
- J5 pad 50: /Mem_addreg6 -> GND
- J5 pad 51: /Mem_addreg7 -> /FLAGS_WE
- J5 pad 52: /Mem_addreg8 -> /PC_INC
- J5 pad 53: /Mem_addreg9 -> /PC_TO_MAR
- J5 pad 54: /Mem_addreg10 -> /SP_INC
- J5 pad 55: /Mem_addreg11 -> /SP_DEC
- J5 pad 56: /Mem_addreg12 -> /RESET_N
- J5 pad 57: /Mem_addreg13 -> /WAIT_N
- J5 pad 58: /Mem_addreg14 -> /IRQ_N
- J5 pad 59: /Mem_addreg15 -> /Unused
- J5 pad 6: J -> /D5
- J5 pad 60: /Mem_addreg16 -> +5V
- J5 pad 61: +5V -> GND
- J5 pad 62: GND -> CLK
- J5 pad 7: A0I -> /D6
- J5 pad 8: A0O -> /D7
- J5 pad 9: A1O -> +5V
- J6 pad 1: MI -> /D0
- J6 pad 10: A1I -> GND
- J6 pad 16: BS -> GND
- J6 pad 2: RI -> /D1
- J6 pad 20: ES1 -> GND
- J6 pad 3: RO -> /D2
- J6 pad 30: SPO -> +5V
- J6 pad 31: HLT -> GND
- J6 pad 32: GND -> /A0
- J6 pad 33: CLK -> /A1
- J6 pad 34: GND -> /A2
- J6 pad 37: Bus C0 -> /A5
- J6 pad 38: Bus C1 -> /A6
- J6 pad 39: Bus C2 -> /A7
- J6 pad 4: CO -> /D3
- J6 pad 40: Bus C3 -> +5V
- J6 pad 41: Bus C4 -> /A8
- J6 pad 42: Bus C5 -> /A9
- J6 pad 43: Bus C6 -> /A10
- J6 pad 44: Bus C7 -> /A11
- J6 pad 45: unconnected-(J6-Pad45) -> /A12
- J6 pad 46: unconnected-(J6-Pad46) -> /A13
- J6 pad 47: unconnected-(J6-Pad47) -> /A14
- J6 pad 48: unconnected-(J6-Pad48) -> /A15
- J6 pad 49: unconnected-(J6-Pad49) -> GND
- J6 pad 5: CE -> /D4
- J6 pad 50: unconnected-(J6-Pad50) -> GND
- J6 pad 51: unconnected-(J6-Pad51) -> /FLAGS_WE
- J6 pad 52: unconnected-(J6-Pad52) -> /PC_INC
- J6 pad 53: unconnected-(J6-Pad53) -> /PC_TO_MAR
- J6 pad 54: unconnected-(J6-Pad54) -> /SP_INC
- J6 pad 55: unconnected-(J6-Pad55) -> /SP_DEC
- J6 pad 56: unconnected-(J6-Pad56) -> /RESET_N
- J6 pad 57: unconnected-(J6-Pad57) -> /WAIT_N
- J6 pad 58: unconnected-(J6-Pad58) -> /IRQ_N
- J6 pad 59: unconnected-(J6-Pad59) -> /Unused
- J6 pad 6: J -> /D5
- J6 pad 60: unconnected-(J6-Pad60) -> +5V
- J6 pad 61: +5V -> GND
- J6 pad 62: GND -> CLK
- J6 pad 7: A0I -> /D6
- J6 pad 8: A0O -> /D7
- J6 pad 9: A1O -> +5V
- J7 pad 1: MI -> /D0
- J7 pad 10: A1I -> GND
- J7 pad 16: BS -> GND
- J7 pad 2: RI -> /D1
- J7 pad 20: ES1 -> GND
- J7 pad 3: RO -> /D2
- J7 pad 30: SPO -> +5V
- J7 pad 31: HLT -> GND
- J7 pad 32: GND -> /A0
- J7 pad 33: CLK -> /A1
- J7 pad 34: GND -> /A2
- J7 pad 37: Bus C0 -> /A5
- J7 pad 38: Bus C1 -> /A6
- J7 pad 39: Bus C2 -> /A7
- J7 pad 4: CO -> /D3
- J7 pad 40: Bus C3 -> +5V
- J7 pad 41: Bus C4 -> /A8
- J7 pad 42: Bus C5 -> /A9
- J7 pad 43: Bus C6 -> /A10
- J7 pad 44: Bus C7 -> /A11
- J7 pad 45: unconnected-(J7-Pad45) -> /A12
- J7 pad 46: unconnected-(J7-Pad46) -> /A13
- J7 pad 47: unconnected-(J7-Pad47) -> /A14
- J7 pad 48: unconnected-(J7-Pad48) -> /A15
- J7 pad 49: unconnected-(J7-Pad49) -> GND
- J7 pad 5: CE -> /D4
- J7 pad 50: unconnected-(J7-Pad50) -> GND
- J7 pad 51: unconnected-(J7-Pad51) -> /FLAGS_WE
- J7 pad 52: unconnected-(J7-Pad52) -> /PC_INC
- J7 pad 53: unconnected-(J7-Pad53) -> /PC_TO_MAR
- J7 pad 54: unconnected-(J7-Pad54) -> /SP_INC
- J7 pad 55: unconnected-(J7-Pad55) -> /SP_DEC
- J7 pad 56: unconnected-(J7-Pad56) -> /RESET_N
- J7 pad 57: unconnected-(J7-Pad57) -> /WAIT_N
- J7 pad 58: unconnected-(J7-Pad58) -> /IRQ_N
- J7 pad 59: unconnected-(J7-Pad59) -> /Unused
- J7 pad 6: J -> /D5
- J7 pad 60: unconnected-(J7-Pad60) -> +5V
- J7 pad 61: +5V -> GND
- J7 pad 62: GND -> CLK
- J7 pad 7: A0I -> /D6
- J7 pad 8: A0O -> /D7
- J7 pad 9: A1O -> +5V
- J8 pad 1: MI -> /D0
- J8 pad 10: A1I -> GND
- J8 pad 16: BS -> GND
- J8 pad 2: RI -> /D1
- J8 pad 20: ES1 -> GND
- J8 pad 3: RO -> /D2
- J8 pad 30: SPO -> +5V
- J8 pad 31: HLT -> GND
- J8 pad 32: GND -> /A0
- J8 pad 33: CLK -> /A1
- J8 pad 34: GND -> /A2
- J8 pad 37: Bus C0 -> /A5
- J8 pad 38: Bus C1 -> /A6
- J8 pad 39: Bus C2 -> /A7
- J8 pad 4: CO -> /D3
- J8 pad 40: Bus C3 -> +5V
- J8 pad 41: Bus C4 -> /A8
- J8 pad 42: Bus C5 -> /A9
- J8 pad 43: Bus C6 -> /A10
- J8 pad 44: Bus C7 -> /A11
- J8 pad 45: /PCount_LED1 -> /A12
- J8 pad 46: /PCount_LED2 -> /A13
- J8 pad 47: /PCount_LED3 -> /A14
- J8 pad 48: /PCount_LED4 -> /A15
- J8 pad 49: /PCount_LED5 -> GND
- J8 pad 5: CE -> /D4
- J8 pad 50: /PCount_LED6 -> GND
- J8 pad 51: /PCount_LED7 -> /FLAGS_WE
- J8 pad 52: /PCount_LED8 -> /PC_INC
- J8 pad 53: /PCount_LED9 -> /PC_TO_MAR
- J8 pad 54: /PCount_LED10 -> /SP_INC
- J8 pad 55: /PCount_LED11 -> /SP_DEC
- J8 pad 56: /PCount_LED12 -> /RESET_N
- J8 pad 57: /PCount_LED13 -> /WAIT_N
- J8 pad 58: /PCount_LED14 -> /IRQ_N
- J8 pad 59: /PCount_LED15 -> /Unused
- J8 pad 6: J -> /D5
- J8 pad 60: /PCount_LED16 -> +5V
- J8 pad 61: +5V -> GND
- J8 pad 62: GND -> CLK
- J8 pad 7: A0I -> /D6
- J8 pad 8: A0O -> /D7
- J8 pad 9: A1O -> +5V
- J9 pad 1: MI -> /D0
- J9 pad 10: A1I -> GND
- J9 pad 16: BS -> GND
- J9 pad 2: RI -> /D1
- J9 pad 20: ES1 -> GND
- J9 pad 3: RO -> /D2
- J9 pad 30: SPO -> +5V
- J9 pad 31: HLT -> GND
- J9 pad 32: GND -> /A0
- J9 pad 33: CLK -> /A1
- J9 pad 34: GND -> /A2
- J9 pad 37: Bus C0 -> /A5
- J9 pad 38: Bus C1 -> /A6
- J9 pad 39: Bus C2 -> /A7
- J9 pad 4: CO -> /D3
- J9 pad 40: Bus C3 -> +5V
- J9 pad 41: Bus C4 -> /A8
- J9 pad 42: Bus C5 -> /A9
- J9 pad 43: Bus C6 -> /A10
- J9 pad 44: Bus C7 -> /A11
- J9 pad 45: /RegB_LED1 -> /A12
- J9 pad 46: /RegB_LED2 -> /A13
- J9 pad 47: /RegB_LED3 -> /A14
- J9 pad 48: /RegB_LED4 -> /A15
- J9 pad 49: /RegB_LED5 -> GND
- J9 pad 5: CE -> /D4
- J9 pad 50: /RegB_LED6 -> GND
- J9 pad 51: /RegB_LED7 -> /FLAGS_WE
- J9 pad 52: /RegB_LED8 -> /PC_INC
- J9 pad 53: /RegB_LED9 -> /PC_TO_MAR
- J9 pad 54: /RegB_LED10 -> /SP_INC
- J9 pad 55: /RegB_LED11 -> /SP_DEC
- J9 pad 56: /RegB_LED12 -> /RESET_N
- J9 pad 57: /RegB_LED13 -> /WAIT_N
- J9 pad 58: /RegB_LED14 -> /IRQ_N
- J9 pad 59: /RegB_LED15 -> /Unused
- J9 pad 6: J -> /D5
- J9 pad 60: /RegB_LED16 -> +5V
- J9 pad 61: +5V -> GND
- J9 pad 62: GND -> CLK
- J9 pad 7: A0I -> /D6
- J9 pad 8: A0O -> /D7
- J9 pad 9: A1O -> +5V
Routing:
- net +5V: track 0.00 -> 355.4 mm
- net CLK: track 0.00 -> 163.3 mm
- net /A2: track 0.00 -> 146.7 mm
- net /A7: track 0.00 -> 146.1 mm
- net /ALU_COUT: track 0.00 -> 146.1 mm
- net /A10: track 0.00 -> 146.0 mm
- net /A11: track 0.00 -> 146.0 mm
- net /A4: track 0.00 -> 146.0 mm
- net /A9: track 0.00 -> 146.0 mm
- net /A3: track 0.00 -> 146.0 mm
- net /ALU_S1: track 0.00 -> 145.9 mm
- net /ALU_S3: track 0.00 -> 145.9 mm
- net /ALU_CIN_N: track 0.00 -> 145.8 mm
- net /D0: track 0.00 -> 145.8 mm
- net /ALU_M: track 0.00 -> 145.8 mm
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