File: Clock/Clock.kicad_sch (KiCad schematic)
At the start: 60 parts, among them J1 Conn buss, J10 Conn_buss, J11 Conn_buss, J12 Conn_buss, J18 Conn_01x02_Pin, J19 Conn_02x04_Top_Bottom, J2 USB4125-GF-A, J3 Fuse-Block, J4 Conn buss, J5 Conn_buss, J6 Conn_buss, J7 Conn_buss, J8 Conn_buss, J9 Conn_buss, SW1 SW_CLK_mono, SW2 SW_Select_Mon/Ast, SW3 SW_SPST, SW4 SW_Select_Oscilator, U1 NE555P, U10 CD74HCT153E, U2 NE555P, U3 NE555P, U4 74LS04, U5 74LS08, U6 CD74HCT14E, U7 NE555P, U9 74HCT244, Y1 ECS-100AX-010

Commit message: Changing to new version of debounce
Parts:
- removed C4, C6: 10 nF, Capacitor_THT:C_Disc_D3.0mm_W2.0mm_P2.50mm, symbol Device:C
- removed C9: 10nF, Capacitor_THT:C_Disc_D3.0mm_W2.0mm_P2.50mm, symbol Device:C
- removed R12: 33, Resistor_THT:R_Axial_DIN0204_L3.6mm_D1.6mm_P5.08mm_Horizontal, symbol Device:R
- removed SW4: SW_Select_Oscilator, Connector_PinHeader_2.54mm:PinHeader_1x03_P2.54mm_Vertical, symbol Switch:SW_SPDT
- removed U2, U3, U7: NE555P, Package_DIP:DIP-8_W7.62mm, symbol Timer:NE555P
- removed U4: 74LS04, Package_DIP:DIP-14_W7.62mm, symbol 74xx:74LS04
- removed U5: 74LS08, Package_DIP:DIP-14_W7.62mm, symbol 74xx:74LS08
- added C4, C6: 1 μF, Capacitor_THT:CP_Radial_D5.0mm_P2.00mm, symbol Device:C_Polarized
- added D2: 1N4001, Diode_THT:D_DO-41_SOD81_P10.16mm_Horizontal, symbol Diode:1N4001
- added D3: LED_Manual, LED_THT:LED_D5.0mm, symbol Device:LED
- added R13: 1k, symbol Device:R
- added R14: 10k, symbol Device:R
- added R4: R, symbol Device:R
- added U2: 74LS00, symbol 74xx:74LS00
- D1: value LED_Turbo -> LED_Run
- D4: value LED_Mon/Ast -> LED_Traice
- D5: value RED -> LED_power
- R10: value 10K -> 1K
- R2: value 100K -> 10K
- SW2: value SW_Select_Mon/Ast -> SW_Select
Connections:
- net CLK_Mon is gone; now on net CLK_Select_Turbo: U6.1 (1A)
- net +5V: now also R14.1; no longer R10.2, U10.16 (VCC), U9.20 (VCC)
- net CLK_Ast: no longer U6.3 (2A)
- net CLK_Select_Mon/Ast: no longer D4.2 (A), U10.14 (S0)
- net CLK_Select_Turbo: no longer D1.2 (A), U10.2 (S1)
- net CLK_Turbo: now also Y1.8 (OUTPUT); no longer U6.5 (3A)
- net GND: now also R10.2, R5.2, R6.2, R13.2; no longer R5.1, R6.1, SW2.2 (B), U10.1 (*1E), U10.15 (*2E), U10.8 (GND), U9.1 (1OE), U9.10 (GND), U9.19 (2OE)
- net at D1.1 (K): now also R6.1; no longer R6.2
- net at R10.1: now also D3.1 (K)
- net at U9.14 (1Y2): no longer U10.3 (1I3)
- net at U9.16 (1Y1): no longer U10.5 (1I1)
- net at U9.2 (1A0): no longer U6.6 (3Y)
- net at U9.4 (1A1): no longer U6.4 (2Y)
- net at U9.6 (1A2): no longer U6.2 (1Y)
- net at R2.1: now also SW1.2, D2.2 (A), R4.1; no longer C8.1
- net CLK_Select_Run: now reaches R3.1, SW2.1 (A)
- net CLK_Select_Run: now also C4.1
- net at D4.1 (K): now also R5.1; no longer R5.2
- net CLK_Select_Traice: now reaches SW2.3 (C)
- net CLK_Select_Traice: now also U6.3 (2A), C6.1, R14.2
- new net: C4.2, C6.2, R13.1, SW2.2 (B)
- new net: U2.12, U2.13, U2.8
- new net: U2.3, U2.4, U2.5
- new net CLK_Manual: C8.1, D2.1 (K), R4.2, U6.5 (3A)
- now unconnected: U10.4 (1I2), U10.6 (1I0), U9.18 (1Y0)
- no-connect marks 24 -> 12
Other:
- note added: "Manual Mode"
- note added: "Run Clock"
- note added: "Selection"
- note removed: "Mono stable 555"
- note removed: "Selection 555"
- note removed: "Selection 555 Turbo"
- note removed: "Turbo Clock"
- moved on the sheet: C8, D1, D4, J18, R2, R3, R5, R6, SW1, SW2, U10, U9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

Commit message: Schimatic with Switch component on the board
Parts:
- removed C11, C15, C16, C17: 100nF, Capacitor_THT:C_Disc_D3.0mm_W2.0mm_P2.50mm, symbol Device:C
- added C13: 470μF, Capacitor_THT:CP_Radial_D8.0mm_P3.50mm, symbol Device:C_Polarized
- added D6: D_TVS, Diode_THT:D_DO-15_P10.16mm_Horizontal, symbol Device:D_TVS
- added J13: Conn_02x08_Top_Bottom, Connector_IDC:IDC-Header_2x08_P2.54mm_Vertical, symbol Connector_Generic:Conn_02x08_Top_Bottom
- added J20: Conn_VCC_GND, Connector_PinHeader_2.54mm:PinHeader_1x02_P2.54mm_Vertical, symbol Connector:Conn_01x02_Pin
- C12: renamed from C10; value 10μF -> 470μF; footprint Capacitor_THT:CP_Radial_D5.0mm_P2.00mm -> Capacitor_THT:CP_Radial_D8.0mm_P3.50mm
- C4: footprint Capacitor_THT:CP_Radial_D5.0mm_P2.00mm -> Capacitor_THT:CP_Radial_D4.0mm_P2.00mm
- C5: renamed from C6; footprint Capacitor_THT:CP_Radial_D5.0mm_P2.00mm -> Capacitor_THT:CP_Radial_D4.0mm_P2.00mm
- D2: footprint Diode_THT:D_DO-41_SOD81_P10.16mm_Horizontal -> Diode_THT:D_DO-41_SOD81_P7.62mm_Horizontal
- J18: value Conn_01x02_Pin -> Conn_CLK
- J19: footprint Connector_PinHeader_2.54mm:PinHeader_2x04_P2.54mm_Vertical -> Connector_IDC:IDC-Header_2x04_P2.54mm_Vertical
- R1, R10, R2, R3, R5, R6, R7, R8, R9: footprint Resistor_THT:R_Axial_DIN0204_L3.6mm_D1.6mm_P5.08mm_Horizontal -> Resistor_THT:R_Axial_DIN0207_L6.3mm_D2.5mm_P7.62mm_Horizontal
- R11: value 5.1K -> 1k; footprint Resistor_THT:R_Axial_DIN0204_L3.6mm_D1.6mm_P5.08mm_Horizontal -> Resistor_THT:R_Axial_DIN0207_L6.3mm_D2.5mm_P7.62mm_Horizontal
- R13, R14, R4: footprint (none) -> Resistor_THT:R_Axial_DIN0207_L6.3mm_D2.5mm_P7.62mm_Horizontal
- SW1: value SW_CLK_mono -> SW_Manual_CLK
- SW3: footprint Connector_PinHeader_2.54mm:PinHeader_1x02_P2.54mm_Vertical -> footprints:CONN2_B2P3-VH_JST
- U2: footprint (none) -> Package_DIP:DIP-14_W7.62mm
- U6: footprint footprints:CD74HCT14E -> Package_DIP:DIP-14_W7.62mm
- U9: footprint (none) -> Package_DIP:DIP-20_W7.62mm
- renumbered C14 to C10, C5 to C11, C7 to C2, C8 to C3, C12 to C6, C2 to C7, C13 to C8, C3 to C9
Connections:
- net CLK_Ast is gone; now on net CLK_Traice: U1.3 (OUT)
- net CLK_Select_Turbo is gone; now on net CLK_Select_Manual: U6.1 (1A)
- net CLK_Turbo is gone; now on net CLK_Run: Y1.8 (OUTPUT)
- net +5V: now also U10.15 (*2E), U10.16 (VCC), U2.14 (VCC), U9.20 (VCC), C13.1, J20.1 (Pin_1)
- net A0: now also J13.1 (Pin_1)
- net A1: now also J13.2 (Pin_2)
- net A10: now also J13.11 (Pin_11)
- net A11: now also J13.12 (Pin_12)
- net A12: now also J13.13 (Pin_13)
- net A13: now also J13.14 (Pin_14)
- net A14: now also J13.15 (Pin_15)
- net A15: now also J13.16 (Pin_16)
- net A2: now also J13.3 (Pin_3)
- net A3: now also J13.4 (Pin_4)
- net A4: now also J13.5 (Pin_5)
- net A5: now also J13.6 (Pin_6)
- net A6: now also J13.7 (Pin_7)
- net A7: now also J13.8 (Pin_8)
- net A8: now also J13.9 (Pin_9)
- net A9: now also J13.10 (Pin_10)
- net CLK: now also U2.6, U6.13 (6A), U9.2 (1A0); no longer J1.62, J10.62, J11.62, J12.62, J18.2 (Pin_2), J4.62, J5.62, J6.62, J7.62, J8.62, J9.62
- net CLK_Run: now also U6.11 (5A)
- net CLK_Select_Run: now also U2.9, U6.3 (2A)
- net CLK_Traice: now also U6.9 (4A)
- net CLK_inv: now also U6.12 (6Y), U9.4 (1A1); no longer J18.1 (Pin_1)
- net GND: now also U10.1 (*1E), U10.8 (GND), U2.7 (GND), U9.1 (1OE), U9.10 (GND), U9.19 (2OE), C13.2, D6.2 (A2), J20.2 (Pin_2)
- net HLT: now also U2.2
- net CLK_Select_Run_inv: now reaches D1.2 (A)
- net CLK_Select_Run_inv: now also U10.14 (S0), U6.4 (2Y)
- net CLK_inv_out: now reaches U9.16 (1Y1)
- net CLK_inv_out: now also J18.1 (Pin_1)
- net CLK_out: now reaches U9.18 (1Y0)
- net CLK_out: now also J1.62, J10.62, J11.62, J12.62, J18.2 (Pin_2), J4.62, J5.62, J6.62, J7.62, J8.62, J9.62
- net CLK_Run_inv: now reaches U6.10 (5Y)
- net CLK_Run_inv: now also U10.4 (1I2)
- net CLK_Select_Manual_inv: now reaches U6.2 (1Y)
- net CLK_Select_Manual_inv: now also D3.2 (A), U10.2 (S1)
- net CLK_Manual_inv: now reaches U6.6 (3Y)
- net CLK_Manual_inv: now also U10.3 (1I3), U10.5 (1I1)
- net CLK_Traice_inv: now reaches U6.8 (4Y)
- net CLK_Traice_inv: now also U10.6 (1I0)
- net at U2.11: now also D4.2 (A)
- net at J2.A9, J2.B9, J3.1: now also D6.1 (A1)
- net at U2.1: now also U10.7 (1Y)
- net CLK_Select_Manual: now reaches U2.10
- net CLK_Select_Manual: now also C5.1, R14.2, SW2.3 (C)
- removed net CLK_Select_Traice: C5.1, R14.2, SW2.3 (C), U6.3 (2A)
- no-connect marks 12 -> 18
Other:
- note added: "Selection LED"
- moved on the sheet: C10, C11, C6, C7, C8, C9, D1, D3, D4, J18, R10, R5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
